Commit message: Package rename.

File: urdf/kinect_v2.urdf.xacro (robot description, xacro)
@@ -1,5 +1,5 @@
 <?xml version="1.0"?>
 <robot name="kinect_v2" xmlns:xacro="http://ros.org/wiki/xacro">
-<xacro:include filename="$(find kinect_v2)/urdf/kinect_v2.gazebo.xacro" />
+<xacro:include filename="$(find kinect_v2_description)/urdf/kinect_v2.gazebo.xacro" />
     <xacro:property name="M_PI" value="3.1415926536" />
     <!-- Kinect2 and mount assembly -->
@@ -19,5 +19,5 @@
                 <origin xyz="0 0 0" rpy="0 0 0" />
                 <geometry>
-                    <mesh filename="package://kinect_v2/meshes/kinect2.stl" />
+                    <mesh filename="package://kinect_v2_description/meshes/kinect2.stl" />
                 </geometry>
                 <material name="">

File: urdf/kinect_v2_standalone.urdf.xacro (robot description, xacro)
@@ -1,9 +1,9 @@
 <?xml version="1.0"?>
 <robot name="kinect_v2_standalone" xmlns:xacro="http://ros.org/wiki/xacro">
-     <xacro:include filename="$(find kinect_v2)/urdf/kinect_v2.urdf.xacro" />
+     <xacro:include filename="$(find kinect_v2_description)/urdf/kinect_v2.urdf.xacro" />
      <link name="root"/>
-    <xacro:kinect_v2  parent="root">
+     <xacro:kinect_v2  parent="root">
         <origin xyz="0 0 0"
                 rpy="0 0 0" />
-    </xacro:kinect_v2>
+     </xacro:kinect_v2>
 </robot>
